File: Hardware/HVPS/HVPS.kicad_sch (KiCad schematic)
At the start: 73 parts, among them J1 Conn_01x01_Socket, J2 Conn_01x01_Socket, J3 Conn_01x01_Socket, J4 Conn_01x01_Socket, J5 Conn_01x01_Socket, J6 Conn_01x01_Socket, J7 Conn_01x01_Socket, J8 Conn_01x01_Socket, J9 Conn_01x01_Socket, Q1 IRF7341PBF, U1 IRS2153D

Commit message: Added scheme of logic board
Parts:
- removed C12, C15, C16, C21, C22: 2200pF, Capacitor_SMD:C_0805_2012Metric, symbol Device:C
- removed D10, D11, D12, D13, D14, D3, D5, D8, D9: SM4007, Diode_SMD:D_MELF, symbol Diode:SM4007
- removed J1, J2, J3, J4, J5, J6, J7, J8, J9: Conn_01x01_Socket, Connector_PinSocket_2.54mm:PinSocket_1x01_P2.54mm_Vertical, symbol Connector:Conn_01x01_Socket
- added C12: 0.1uF, symbol Device:C_Small
- added C23: C_Small, symbol Device:C_Small
- added D1: SS24, Diode_SMD:D_SMA, symbol Diode:SS24
- added J1: Conn_01x08_Pin, Connector_RJ:RJ9_Evercom_5301-440xxx_Horizontal, symbol Connector:Conn_01x08_Pin
- added J10: Conn_01x14_Pin, symbol Connector:Conn_01x14_Pin
- added L1: L, Inductor_SMD:L_7.3x7.3_H4.5, symbol Device:L
- added PS1: MEE1S0303SC, Converter_DCDC:Converter_DCDC_Murata_MEE1SxxxxSC_THT, symbol Converter_DCDC:MEE1S0303SC
- added Q2: 2N7002, Package_TO_SOT_SMD:SOT-23, symbol Transistor_FET:2N7002
- added R29: 100k, Resistor_SMD:R_1210_3225Metric, symbol Device:R
- added R30, R31, R32: 10k, Resistor_SMD:R_0805_2012Metric, symbol Device:R
- added U10: AOZ1280CI, Package_TO_SOT_SMD:SOT-23-6, symbol Regulator_Switching:AOZ1280CI
- added U11: DAC6311xDCK, Package_TO_SOT_SMD:SOT-363_SC-70-6, symbol Analog_DAC:DAC6311xDCK
- added U13: LM6172, Package_SO:SOIC-8_3.9x4.9mm_P1.27mm, symbol Amplifier_Operational:LM6172
- added U14: ISO7762DBQ, Package_SO:SSOP-16_3.9x4.9mm_P0.635mm, symbol Isolator:ISO7762DBQ
- added U2, U3: MCP4922-ESL, Package_SO:SOIC-14_3.9x8.7mm_P1.27mm, symbol Analog_DAC:MCP4922-ESL
- added U4, U5: OP279, symbol Amplifier_Operational:OP279
- added U7: ADS7886xxDBV, Package_TO_SOT_SMD:SOT-23-6, symbol Analog_ADC:ADS7886xxDBV
- added U8: LM397, Package_TO_SOT_SMD:SOT-23-5, symbol Comparator:LM397
- added U9: ISO7761FDBQ, Package_SO:SSOP-16_3.9x4.9mm_P0.635mm, symbol Isolator:ISO7761FDBQ
- C10, C13, C14, C6, C7, C8: value 2200pF -> 47nF; Part Name (none) -> C2225C473KFRACTU; Voltage 1000V -> 1500V
- C11: value 2200pF -> 10uF; Voltage 1000V -> 25V
- C4: value 4700pF -> 100nF; footprint Capacitor_SMD:C_0805_2012Metric -> Capacitor_SMD:C_2220_5750Metric; Part Name (none) -> GRM55DR73A104KW01L; Voltage 500V -> 1000V
- C5: value 2200pF -> 4.7uF; Voltage 1000V -> 25V
- R24, R25: value 3M3 -> 10M
- R26: value 3M3 -> 4.7k; footprint Resistor_SMD:R_2512_6332Metric -> Resistor_SMD:R_0805_2012Metric
- R5: footprint Resistor_SMD:R_0805_2012Metric -> Resistor_SMD:R_1210_3225Metric
- R6, R8: value 3M3 -> 36k; footprint Resistor_SMD:R_2512_6332Metric -> Resistor_SMD:R_0805_2012Metric
- R7: value 3M3 -> 1k; footprint Resistor_SMD:R_2512_6332Metric -> Resistor_SMD:R_0805_2012Metric
- R9: value 100k -> 36k
Connections:
- net GNDA: now also C13.1, C14.1, C7.1, R7.1, R8.1, PS1.3 (-Vout), U14.9 (GND2), U9.9 (GND2); no longer C1.2, C2.1, C20.2, C3.2, C5.1, R10.2, R3.2, U1.4 (COM), U1.6 (VS)
- net at C13.2: now also C8.1
- net at R25.2: now also R24.1; no longer R26.1
- net at R5.1: now also C6.2, D4.2 (A); no longer R26.2
- net GND: now reaches C11.1
- net GND: now also C1.2, C2.1, C3.2, C5.1, R3.2, U1.4 (COM), U1.6 (VS), D1.2 (A), PS1.1 (-Vin), Q2.2 (S), R31.2, U10.2 (GND), U14.8 (GND1), U9.8 (GND1)
- net at C8.2: now also C10.2, R24.2, R5.2, R29.1; no longer C13.1
- net at C1.1, R4.2, U1.3 (CT): now also Q2.3 (D)
- net +5V renamed +12V
- net +12V: now also C5.2, U10.4 (EN), U10.5 (VIN); no longer C3.1, TR1.2
- net Cathode: no longer names the net of C9.1, R19.1
- net Cathode: now also R7.2, U5.5 (+); no longer R9.2
- new net: C12.2, D1.1 (K), L1.1, U10.6 (LX)
- new net: C11.2, C3.1, L1.2, R30.1, TR1.2
- new net: C12.1, U10.1 (BST)
- new net: U5.6 (-), U5.7, U8.3 (+)
- new net: U4.1, U4.2 (-), U7.3 (VIN)
- new net: U14.15 (OUTA), U7.4 (SCLK)
- new net: U14.11 (INE), U7.5 (SDO)
- new net: U14.14 (OUTB), U7.6 (~{CS})
- new net: U2.8 (~{LDAC}), U3.8 (~{LDAC}), U9.11 (OUTE)
- new net: U3.3 (~{CS}), U9.12 (OUTD)
- new net: U2.3 (~{CS}), U9.13 (OUTC)
- new net: U2.4 (SCK), U3.4 (SCK), U9.14 (OUTB)
- new net: U2.5 (SDI), U3.5 (SDI), U9.15 (OUTA)
- new net: J1.1 (Pin_1), U11.3 (DIN), U9.2 (INA)
- new net: J1.2 (Pin_2), U11.2 (SCLK), U9.3 (INB)
- new net: J1.3 (Pin_3), U9.4 (INC)
- new net: J1.4 (Pin_4), U9.5 (IND)
- new net: J1.5 (Pin_5), U9.6 (INE)
- new net: Q2.1 (G), U9.7 (OUTF)
- new net: R8.2, R9.1, U8.1 (-)
- new net: R25.1, R6.2, U4.3 (+)
- new net: C10.1, C14.2
- new net: J1.6 (Pin_6), U14.3 (INB)
- new net: J1.7 (Pin_7), U14.7 (OUTF)
- new net: J1.8 (Pin_8), U11.1 (~{SYNC})
- new net: R30.2, R31.1, R32.2, U10.3 (FB)
- new net: C7.2, D4.1 (K), D6.2 (A)
- new net: C20.2, J10.2 (Pin_2), R10.2, R29.2
- new net: R32.1, U11.6 (VOUT)
- new net: R26.1, U14.10 (INF), U8.4
Other:
- note added: "12V * 62.5 = 750V"
- note added: "500V * 3 = 1500V"
- note added: "5V...11V"
- note added: "600V * 3 = 1800V"
- note added: "750V * 3 = 2250V"
- note added: "8V * 62.5 = 500V"
- note added: "9.6V * 62.5 = 600V"
- note added: "Anode 1,3"
- note added: "Anode 2 (Focus)"
- note added: "Cathode"
- note added: "Def X1"
- note added: "Def X2"
- note added: "Def Y1"
- note added: "Def Y2"
- note added: "Grid"
- note added: "Heater 1"
- note added: "Heater 2"
- note added: "Зона высокого напряжения"
- note added: "К ЭЛТ"
- note added: "Монитор напряжения"
- note added: "Монитор тока"
- note added: "Уставка ВВ напряжения"
- moved on the sheet: C1, C17, C18, C19, C2, C20, C3, C4, C9, D4, D6, D7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
