File: Hardware/Logic/Logic.kicad_sch (KiCad schematic)
At the start: 11 parts, among them Q1 DMG2305UX, U1 MCP4922-ESL, U2 MCP4922-ESL, U3 LM6172

Commit message: Added scheme of logic board
Parts:
- removed U3: LM6172, Package_SO:SOIC-8_3.9x4.9mm_P1.27mm, symbol Amplifier_Operational:LM6172
- added BT1: Battery, Battery:Battery_Panasonic_CR2032-HFN_Horizontal_CircularHoles, symbol Device:Battery
- added C15, C16, C21, C22, C29: 0.1uF, Capacitor_SMD:C_0805_2012Metric, symbol Device:C_Small
- added C26, C27, C28: 10uF, Capacitor_SMD:C_0805_2012Metric, symbol Device:C_Small
- added D2: LED, LED_SMD:LED_0805_2012Metric, symbol Device:LED
- added D3: BAT54A, Package_TO_SOT_SMD:SOT-23, symbol Diode:BAT54A
- added D5: SS24, Diode_SMD:D_SMA, symbol Diode:SS24
- added FB1, FB2: FerriteBead_Small, Inductor_SMD:L_0805_2012Metric, symbol Device:FerriteBead_Small
- added J2: USB_C_Receptacle, Connector_USB:USB_C_Receptacle_GCT_USB4115-03-C, symbol Connector:USB_C_Receptacle
- added J3: Conn_01x05_Socket, symbol Connector:Conn_01x05_Socket
- added J4: SD_Card_Receptacle, Connector_Card:SD_TE_2041021, symbol Connector:SD_Card_Receptacle
- added R33, R34, R36, R37, R38, R45: 10k, Resistor_SMD:R_0805_2012Metric, symbol Device:R
- added R35, R43, R44: 1k, Resistor_SMD:R_0805_2012Metric, symbol Device:R
- added R39, R40: 4.7k, Resistor_SMD:R_0805_2012Metric, symbol Device:R
- added R41, R42: 5.1k, Resistor_SMD:R_0805_2012Metric, symbol Device:R
- added SW1: SW_Omron_B3FS, Button_Switch_SMD:SW_SPST_Omron_B3FS-100xP, symbol Switch:SW_Omron_B3FS
- added U12: ESP32-S3-WROOM-1, RF_Module:ESP32-S3-WROOM-1, symbol RF_Module:ESP32-S3-WROOM-1
- added U15: MAX98357A, Package_DFN_QFN:TQFN-16-1EP_3x3mm_P0.5mm_EP1.23x1.23mm, symbol Audio:MAX98357A
- added U16: DS3231M, Package_SO:SOIC-16W_7.5x10.3mm_P1.27mm, symbol Timer_RTC:DS3231M
- added U17: SCD41-D-R2, Sensor:Sensirion_SCD4x-1EP_10.1x10.1mm_P1.25mm_EP4.8x4.8mm, symbol Sensor_Gas:SCD41-D-R2
- added U18: VL53L0CXV0DH1, Sensor_Distance:ST_VL53L1x, symbol Sensor_Distance:VL53L0CXV0DH1
- added U19, U20: LM4040DBZ-2.0, Package_TO_SOT_SMD:SOT-23, symbol Reference_Voltage:LM4040DBZ-2.0
- added U6: PC817, Package_DIP:DIP-4_W7.62mm, symbol Isolator:PC817
- C24: value 0.1uF -> 100uF
- C25: value 10uF -> 100uF
Connections:
- net +3V3: now also C16.1, C21.1, C22.1, FB1.2, FB2.2, J4.4 (VDD), R33.1, R34.1, R35.1, R36.1, R37.1, R38.1, R39.2, R40.2, R43.2, R44.2, R45.1, U12.2 (3V3), U16.2 (VCC), U17.19 (VDD), U17.7 (VDD), U18.11 (AVDD); no longer C1.1, C23.1, C25.1, U1.1 (VDD), U2.1 (VDD)
- net GND: now also BT1.2 (-), C15.2, C16.2, C21.2, C22.2, C26.2, C27.2, C28.2, C29.2, J2.A1 (GND), J2.A12 (GND), J2.B1 (GND), J2.B12 (GND), J4.3 (VSS), J4.6 (VSS), SW1.2, U12.1 (GND), U12.40 (GND), U12.41 (GND), U15.11 (GND), U15.15 (GND), U15.17 (PAD), U15.3 (GND), U16.10 (GND), U16.11 (GND), U16.12 (GND), U16.13 (GND), U16.5 (GND), U16.6 (GND), U16.7 (GND), U16.8 (GND), U16.9 (GND), U17.20 (GND), U17.21 (GND), U17.6 (GND), U18.12 (GND), U18.3 (GND), U18.4 (GND), U18.6 (GND), U19.2 (A), U20.2 (A), U6.3
- net at U1.11 (VrefB): now also U1.13 (VrefA), C27.1, C28.1, R43.1, U19.1 (K)
- net at U1.3 (~{CS}): now also A1.6 (GPIO4); no longer A1.24 (GPIO18)
- net at U1.4 (SCK), U2.4 (SCK): now also A1.4 (GPIO2); no longer A1.22 (GPIO17)
- net at U1.5 (SDI), U2.5 (SDI): now also A1.5 (GPIO3); no longer A1.21 (GPIO16)
- net at U1.8 (~{LDAC}), U2.8 (~{LDAC}): now also A1.9 (GPIO6); no longer A1.25 (GPIO19)
- net at U2.11 (VrefB): now also C23.1, U2.13 (VrefA), C26.1, R44.1, U20.1 (K)
- net at U2.3 (~{CS}): now also A1.7 (GPIO5); no longer A1.26 (GPIO20)
- net at A1.1 (GPIO0): now also U12.38 (IO2)
- net at A1.15 (GPIO11): now also R33.2, U6.4
- net at A1.2 (GPIO1): now also U12.39 (IO1)
- net VEE renamed +5V
- net +5V: now also C25.1, C29.1, D5.2 (A), U15.7 (VDD), U15.8 (VDD)
- new net: C15.1, FB2.1, U1.1 (VDD)
- new net: R45.2, U18.5 (XSHUT)
- new net: C1.1, FB1.1, U2.1 (VDD)
- new net: R38.2, U16.4 (~{RST})
- new net: D2.2 (A), R35.2
- new net: R37.2, SW1.1, U12.27 (IO0)
- new net: R40.1, U12.20 (IO12), U16.16 (SCL), U17.9 (SCL), U18.10 (SCL)
- new net: D2.1 (K), U12.23 (IO21)
- new net: U12.22 (IO14), U18.7 (GPIO1)
- new net: R39.1, U12.19 (IO11), U16.15 (SDA), U17.10 (SDA), U18.9 (SDA)
- new net: J3.4 (Pin_4), R34.2
- new net: J2.A5 (CC1), R41.2
- new net: U12.17 (IO9), U15.1 (DIN)
- new net: U12.12 (IO8), U15.14 (LRCLK)
- new net: U12.7 (IO7), U15.16 (BCLK)
- new net: U12.33 (IO40), U15.2 (GAIN_SLOT)
- new net: U12.18 (IO10), U15.4 (~{SD_MODE})
- new net: D3.1, U16.14 (VBAT)
- new net: BT1.1 (+), D3.3
- new net: J2.A6 (D+), J2.B6 (D+), U12.14 (USB_D+)
- new net: J2.A7 (D-), J2.B7 (D-), U12.13 (USB_D-)
- new net: J2.B5 (CC2), R42.2
- new net: U12.21 (IO13), U16.3 (~{INT}/SQW)
- new net: J3.3 (Pin_3), U12.10 (IO17)
- new net: J3.5 (Pin_5), U12.11 (IO18)
- new net: J4.5 (CLK), U12.15 (IO3)
- new net: R36.2, U12.3 (EN)
- new net: J4.2 (CMD), U12.4 (IO4)
- new net: J4.7 (DAT0), U12.5 (IO5)
- new net: J4.1 (CD/DAT3), U12.6 (IO6)
- new net: J3.1 (Pin_1), U12.8 (IO15)
- new net: J3.2 (Pin_2), U12.9 (IO16)
- new net Vbus: D5.1 (K), J2.A4 (VBUS), J2.A9 (VBUS), J2.B4 (VBUS), J2.B9 (VBUS), R41.1, R42.1
Other:
- note added: "Button MODE"
- note added: "Encoder A"
- note added: "Encoder B"
- note added: "Encoder BTN"
- moved on the sheet: A1, C1, C23, Q1, R27, R28, U1, U2
